File: ai03-pcb-practice.kicad_sch (KiCad schematic)
At the start: 0 parts

Commit message: Schematic
Parts:
- added C1, C2, C3: .01uF, Capacitor_SMD:C_0805_2012Metric, symbol Device:C_Small
- added C4, C5: 22pF, Capacitor_SMD:C_0805_2012Metric, symbol Device:C_Small
- added C6: 10uF, Capacitor_SMD:C_0805_2012Metric, symbol Device:C_Small
- added C7: 1uF, Capacitor_SMD:C_0805_2012Metric, symbol Device:C_Small
- added D1, D2, D3, D4: SOD-123, Diode_SMD:D_SOD-123, symbol Device:D_Small
- added F1: 500mA, Fuse:Fuse_1206_3216Metric, symbol Device:Polyfuse_Small
- added MX1, MX2, MX3, MX4: MX-NoLED, MX_Alps_Hybrid:MX-1U, symbol MX_Alps_Hybrid:MX-NoLED
- added R1, R2: 22, Resistor_SMD:R_0805_2012Metric, symbol Device:R_Small
- added R3, R4: 10k, Resistor_SMD:R_0805_2012Metric, symbol Device:R_Small
- added SW1: SW_Push, random-keyboard-parts:SKQG-1155865, symbol Switch:SW_Push
- added U1: ATmega32U4-A, Package_QFP:TQFP-44_10x10mm_P0.8mm, symbol MCU_Microchip_ATmega:ATmega32U4-A
- added USB1: Molex-0548190589, random-keyboard-parts:Molex-0548190589, symbol random-keyboard-parts:Molex-0548190589
- added Y1: 16MHz, Crystal:Crystal_SMD_3225-4Pin_3.2x2.5mm, symbol Device:Crystal_GND24_Small
Connections:
- new net: D2.2 (A), MX2.2 (ROW)
- new net: R2.1, U1.4 (D+)
- new net: R3.2, SW1.2, U1.13 (~{RESET})
- new net: C5.1, U1.16 (XTAL2), Y1.3
- new net: C4.2, U1.17 (XTAL1), Y1.1
- new net: R1.1, U1.3 (D-)
- new net: R4.1, U1.33 (~{HWB}/PE2)
- new net: C7.1, U1.6 (UCAP)
- new net: D3.2 (A), MX3.2 (ROW)
- new net: D4.2 (A), MX4.2 (ROW)
- new net: D1.2 (A), MX1.2 (ROW)
- new net +5V: C1.1, C2.1, C3.1, C6.1, F1.2, R3.1, U1.14 (VCC), U1.2 (UVCC), U1.24 (AVCC), U1.34 (VCC), U1.44 (AVCC), U1.7 (VBUS)
- new net COL0: D2.1 (K), D4.1 (K), MX2.1 (COL), U1.27 (PD7), U1.29 (PB5)
- new net COL1: MX3.1 (COL), MX4.1 (COL), U1.28 (PB4)
- new net D+: R2.2, USB1.3 (D+)
- new net D-: R1.2, USB1.4 (D-)
- new net GND: C1.2, C2.2, C3.2, C4.1, C5.2, C6.2, C7.2, R4.2, SW1.1, U1.15 (GND), U1.23 (GND), U1.35 (GND), U1.43 (GND), U1.5 (UGND), USB1.1 (GND), Y1.2, Y1.4
- new net ROW1: D3.1 (K), U1.30 (PB6)
- new net VCC: F1.1, USB1.5 (VBUS)

Commit message: Progress
Parts:
- MX1, MX2, MX3, MX4: footprint MX_Alps_Hybrid:MX-1U -> MX_Alps_Hybrid:MX-1U-NoLED
Connections:
- net COL0: now also MX1.1 (COL)
- net ROW1: now also D1.1 (K)
Other:
- moved on the sheet: D3, MX1, MX3
