File: ai03-pcb-practice.kicad_pcb (KiCad board)
At the start: 2 copper layers, 74.6 x 38.1 mm, 24 parts, among them SW1 SW_Push, U1 ATmega32U4-A, Y1 16MHz

Commit message: Fixing Errors
Parts:
- C1, C2, C3, C4, C5, C6, C7, D1, D2, D3, D4, F1, R1, R2, R3, R4, SW1, U1, USB1, Y1: moved to B.Cu
- MX1, MX2, MX3, MX4: moved to F.Cu
- moved Y1 19.9 mm to (72.4, 106.9), turned to 180 degrees
- moved C4 19.8 mm to (76.2, 107.0)
- moved C5 19.8 mm to (68.6, 107.0)
- moved C6 17.8 mm to (63.5, 121.9), turned to 90 degrees
- moved C1 17.8 mm to (67.0, 125.1)
- moved R3 16.6 mm to (64.5, 108.6)
- moved C3 15.8 mm to (77.2, 125.1), turned to 180 degrees
- moved F1 12.2 mm to (50.8, 113.8), turned to -90 degrees
- moved R4 7.80 mm to (81.3, 122.3)
- moved C2 6.07 mm to (81.3, 111.8), turned to 90 degrees
- moved C7 5.38 mm to (63.5, 114.6), turned to -90 degrees
- moved R2 4.10 mm to (55.9, 108.9), turned to 90 degrees
- moved R1 3.43 mm to (53.2, 108.9), turned to 90 degrees
- moved SW1 3.17 mm to (57.1, 127.6), turned to 180 degrees
- moved USB1 1.75 mm to (54.6, 99.3)
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Routing:
- net COL0: track 0.00 -> 77.2 mm, vias 0 -> 2
- net ROW1: track 0.00 -> 53.3 mm
- net COL1: track 0.00 -> 48.2 mm
- net +5V: track 57.0 -> 101.1 mm, vias 0 -> 6
- net GND: track 75.5 -> 113.4 mm, vias 0 -> 6
- net unconnected-(USB1-Pad6): track 0.00 -> 25.2 mm
- net Net-(R3-Pad2): track 19.8 -> 29.4 mm, vias 0 -> 2
- net Net-(C4-Pad2): track 15.7 -> 6.64 mm, vias 2 -> 0
- net Net-(D2-Pad2): track 0.00 -> 6.95 mm
- net Net-(D3-Pad2): track 0.00 -> 6.82 mm
- net Net-(D4-Pad2): track 0.00 -> 6.62 mm
- net Net-(D1-Pad2): track 0.00 -> 6.29 mm
- net Net-(R1-Pad1): track 11.2 -> 17.4 mm
- net D+: track 10.4 -> 4.74 mm
- net VCC: track 4.31 -> 9.49 mm
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Other:
- outline, holes or cut-outs redrawn

Commit message: Yup
Routing:
- added copper zone on B.Cu, net GND
- added copper zone on F.Cu, net GND
Changed lines of the file:
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@@
   (segment (start 120.65 105.50625) (end 118.0625 105.50625) (width 0.254) (layer "B.Cu") (net 43))
   (segment (start 118.0625 105.50625) (end 115.2125 102.65625) (width 0.254) (layer "B.Cu") (net 43))
+  (zone (net 2) (net_name "GND") (layers F&B.Cu) (hatch edge 0.508)
+    (connect_pads (clearance 0.508))
+    (min_thickness 0.254) (filled_areas_thickness no)
+    (fill yes (thermal_gap 0.508) (thermal_bridge_width 0.508))
+    (polygon
+      (pts
+        (xy 84.1375 135.73125)
+        (xy 47.625 135.73125)
+        (xy 47.625 97.63125)
+        (xy 84.1375 97.63125)
+      )
+    )
+  )
 )
